File: 1.PCB_PARALYSIS_ASSIST/Balaji_Paralysis_Assist/Paralysis_Assist_v1.brd (EAGLE design)
At the start: 106.7 x 100 mm, 24 parts, among them IC2 7805TV, U1 ZC563900

Commit message: added image
Parts:
- moved D1 22.3 mm to (14.7, 83.1)
- moved R1 18.5 mm to (18.2, 80.8)
- moved LM386 3.18 mm to (73.5, 92.7)
Routing:
- net GND: track 360.0 -> 381.4 mm
- net 5V: track 218.6 -> 223.6 mm
- net AUDIO_OUT: track 74.4 -> 71.3 mm
- net 9_IN: track 95.2 -> 92.1 mm
- net SCK: track 101.9 -> 103.8 mm
- net N$3: track 2.46 -> 3.46 mm
- net 3V3: track 62.3 -> 63.0 mm
- net RXNANO: track 37.5 -> 38.2 mm
- net MISO: track 48.3 -> 48.9 mm
Other:
- board size 106.7 x 100 mm -> 106.8 x 100.6 mm
- board text added: "Paralysis Assist"
- board text removed: "P_ASSIST"

Commit message: pcb changes
Connections:
- net CS_DISP: now also JP2.3, NANO.13; no longer JP2.2, NANO.14
- net MISO: now also JP2.1, NANO.15; no longer JP2.8, NANO.8
- net MOSI: now also JP2.2, NANO.14; no longer JP2.3, NANO.13
- net RST: now also JP2.8, NANO.8; no longer JP2.1, NANO.15
Routing:
- net RST: track 47.0 -> 27.7 mm
- net MISO: track 48.9 -> 41.8 mm
- net CS_DISP: track 59.8 -> 57.3 mm
- net MOSI: track 140.7 -> 140.0 mm
Changed lines of the file:
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@@
 <drawing>
 <settings>
-<setting alwaysvectorfont="yes"/>
+<setting alwaysvectorfont="no"/>
 <setting verticaltext="up"/>
 </settings>
 <grid distance="5" unitdist="mil" unit="mil" style="lines" multiple="1" display="no" altdistance="5" altunitdist="mil" altunit="mil"/>
 <layers>
-<layer number="1" name="Top" color="4" fill="1" visible="no" active="yes"/>
+<layer number="1" name="Top" color="4" fill="1" visible="yes" active="yes"/>
 <layer number="2" name="Route2" color="16" fill="1" visible="no" active="no"/>
 <layer number="3" name="Route3" color="17" fill="1" visible="no" active="no"/>
@@
 <layer number="17" name="Pads" color="2" fill="1" visible="yes" active="yes"/>
 <layer number="18" name="Vias" color="2" fill="1" visible="yes" active="yes"/>
-<layer number="19" name="Unrouted" color="6" fill="1" visible="no" active="yes"/>
+<layer number="19" name="Unrouted" color="6" fill="1" visible="yes" active="yes"/>
 <layer number="20" name="Dimension" color="24" fill="1" visible="yes" active="yes"/>
-<layer number="21" name="tPlace" color="7" fill="1" visible="no" active="yes"/>
-<layer number="22" name="bPlace" color="7" fill="1" visible="no" active="yes"/>
-<layer number="23" name="tOrigins" color="15" fill="1" visible="no" active="yes"/>
-<layer number="24" name="bOrigins" color="15" fill="1" visible="no" active="yes"/>
-<layer number="25" name="tNames" color="7" fill="1" visible="no" active="yes"/>
-<layer number="26" name="bNames" color="7" fill="1" visible="no" active="yes"/>
+<layer number="21" name="tPlace" color="7" fill="1" visible="yes" active="yes"/>
+<layer number="22" name="bPlace" color="7" fill="1" visible="yes" active="yes"/>
+<layer number="23" name="tOrigins" color="15" fill="1" visible="yes" active="yes"/>
+<layer number="24" name="bOrigins" color="15" fill="1" visible="yes" active="yes"/>
+<layer number="25" name="tNames" color="7" fill="1" visible="yes" active="yes"/>
+<layer number="26" name="bNames" color="7" fill="1" visible="yes" active="yes"/>
 <layer number="27" name="tValues" color="7" fill="1" visible="no" active="yes"/>
 <layer number="28" name="bValues" color="7" fill="1" visible="no" active="yes"/>
@@
 <layer number="37" name="tTest" color="7" fill="1" visible="no" active="yes"/>
 <layer number="38" name="bTest" color="7" fill="1" visible="no" active="yes"/>
-<layer number="39" name="tKeepout" color="4" fill="11" visible="no" active="yes"/>
-<layer number="40" name="bKeepout" color="1" fill="11" visible="no" active="yes"/>
-<layer number="41" name="tRestrict" color="4" fill="10" visible="no" active="yes"/>
-<layer number="42" name="bRestrict" color="1" fill="10" visible="no" active="yes"/>
+<layer number="39" name="tKeepout" color="4" fill="11" visible="yes" active="yes"/>
+<layer number="40" name="bKeepout" color="1" fill="11" visible="yes" active="yes"/>
+<layer number="41" name="tRestrict" color="4" fill="10" visible="yes" active="yes"/>
+<layer number="42" name="bRestrict" color="1" fill="10" visible="yes" active="yes"/>
 <layer number="43" name="vRestrict" color="2" fill="10" visible="no" active="yes"/>
 <layer number="44" name="Drills" color="7" fill="1" visible="no" active="yes"/>
@@
 <layer number="49" name="Reference" color="7" fill="1" visible="no" active="yes"/>
 <layer number="50" name="dxf" color="7" fill="1" visible="no" active="no"/>
-<layer number="51" name="tDocu" color="7" fill="1" visible="no" active="yes"/>
-<layer number="52" name="bDocu" color="7" fill="1" visible="no" active="yes"/>
+<layer number="51" name="tDocu" color="7" fill="1" visible="yes" active="yes"/>
+<layer number="52" name="bDocu" color="7" fill="1" visible="yes" active="yes"/>
 <layer number="53" name="tGND_GNDA" color="7" fill="9" visible="no" active="no"/>
 <layer number="54" name="bGND_GNDA" color="1" fill="9" visible="no" active="no"/>
@@
 <contactref element="SD_CARD" pad="4"/>
 <contactref element="DISP" pad="5"/>
-<contactref element="NANO" pad="13"/>
-<contactref element="JP2" pad="3"/>
-<wire x1="52.324" y1="28.575" x2="45.974" y2="28.575" width="0.635" layer="16"/>
 <wire x1="71.374" y1="71.755" x2="71.374" y2="66.675" width="0.635" layer="16"/>
 <wire x1="68.834" y1="64.135" x2="66.294" y2="64.135" width="0.635" layer="16"/>
@@
 <wire x1="62.484" y1="60.325" x2="62.484" y2="34.925" width="0.635" layer="16"/>
 <wire x1="62.484" y1="34.925" x2="56.134" y2="28.575" width="0.635" layer="16"/>
-<wire x1="56.134" y1="28.575" x2="52.324" y2="28.575" width="0.635" layer="16"/>
 <wire x1="71.374" y1="66.675" x2="68.834" y2="64.135" width="0.635" layer="16"/>
 <via x="100.203" y="12.954" extent="1-16" drill="1.016"/>
@@
 <wire x1="89.154" y1="5.715" x2="92.8398" y2="2.0292" width="0.635" layer="16"/>
 <wire x1="101.854" y1="11.303" x2="101.854" y2="3.2385" width="0.635" layer="1"/>
-<wire x1="52.324" y1="28.575" x2="54.864" y2="28.575" width="0.635" layer="16"/>
 <wire x1="70.485" y1="12.954" x2="100.203" y2="12.954" width="0.635" layer="16"/>
-<wire x1="54.864" y1="28.575" x2="70.485" y2="12.954" width="0.635" layer="16"/>
+<wire x1="70.485" y1="12.954" x2="54.864" y2="28.575" width="0.635" layer="16"/>
+<contactref element="NANO" pad="14"/>
+<contactref element="JP2" pad="2"/>
+<wire x1="52.324" y1="26.035" x2="45.974" y2="26.035" width="0.635" layer="16"/>
+<wire x1="56.134" y1="28.575" x2="54.864" y2="28.575" width="0.635" layer="16"/>
+<wire x1="54.864" y1="28.575" x2="53.848" y2="27.559" width="0.635" layer="16"/>
+<wire x1="53.848" y1="27.559" x2="53.848" y2="26.162" width="0.635" layer="16"/>
+<wire x1="53.848" y1="26.162" x2="53.721" y2="26.035" width="0.635" layer="16"/>
+<wire x1="53.721" y1="26.035" x2="52.324" y2="26.035" width="0.635" layer="16"/>
 </signal>
 <signal name="MISO">
-<contactref element="NANO" pad="8"/>
-<contactref element="JP2" pad="8"/>
 <contactref element="SD_CARD" pad="5"/>
-<wire x1="52.324" y1="41.275" x2="45.974" y2="41.275" width="0.635" layer="16"/>
 <wire x1="60.706" y1="42.545" x2="59.436" y2="41.275" width="0.635" layer="16"/>
-<wire x1="52.324" y1="41.275" x2="59.436" y2="41.275" width="0.635" layer="16"/>
 <wire x1="60.706" y1="42.545" x2="60.706" y2="61.595" width="0.635" layer="16"/>
 <wire x1="60.706" y1="61.595" x2="65.786" y2="66.675" width="0.635" layer="16"/>
@@
 <wire x1="67.564" y1="66.675" x2="68.834" y2="67.945" width="0.635" layer="16"/>
 <wire x1="68.834" y1="67.945" x2="68.834" y2="71.755" width="0.635" layer="16"/>
+<contactref element="NANO" pad="15"/>
+<contactref element="JP2" pad="1"/>
+<wire x1="52.324" y1="23.495" x2="45.974" y2="23.495" width="0.635" layer="16"/>
+<wire x1="52.324" y1="23.495" x2="59.436" y2="41.275" width="0" layer="19" extent="16-16"/>
 </signal>
 <signal name="TXNANO">
@@
 </signal>
 <signal name="RST">
-<contactref element="NANO" pad="15"/>
-<contactref element="JP2" pad="1"/>
 <contactref element="DISP" pad="4"/>
-<wire x1="52.324" y1="23.495" x2="45.974" y2="23.495" width="0.635" layer="16"/>
-<wire x1="52.324" y1="23.495" x2="53.594" y2="23.495" width="0.635" layer="16"/>
-<wire x1="53.594" y1="23.495" x2="56.134" y2="20.955" width="0.635" layer="16"/>
 <via x="56.134" y="20.955" extent="1-16" drill="1.016"/>
-<wire x1="56.134" y1="20.955" x2="66.294" y2="10.795" width="0.635" layer="1"/>
 <wire x1="66.294" y1="10.795" x2="73.279" y2="10.795" width="0.635" layer="1"/>
 <via x="73.279" y="10.795" extent="1-16" drill="1.016"/>
 <wire x1="73.279" y1="10.795" x2="84.074" y2="10.795" width="0.635" layer="16"/>
 <wire x1="84.074" y1="10.795" x2="86.614" y2="8.255" width="0.635" layer="16"/>
+<contactref element="NANO" pad="8"/>
+<contactref element="JP2" pad="8"/>
+<wire x1="52.324" y1="41.275" x2="45.974" y2="41.275" width="0.635" layer="16"/>
+<wire x1="56.134" y1="20.955" x2="52.324" y2="41.275" width="0" layer="19" extent="1-1"/>
+<wire x1="66.294" y1="10.795" x2="56.134" y2="20.955" width="0" layer="19" extent="1-1"/>
 </signal>
 <signal name="TEMP">
@@
 <signal name="CS_DISP">
 <contactref element="DISP" pad="3"/>
-<contactref element="NANO" pad="14"/>
-<contactref element="JP2" pad="2"/>
-<wire x1="52.324" y1="26.035" x2="45.974" y2="26.035" width="0.635" layer="16"/>
-<wire x1="52.324" y1="26.035" x2="54.864" y2="26.035" width="0.635" layer="16"/>
 <wire x1="63.119" y1="17.78" x2="63.119" y2="11.303" width="0.635" layer="16"/>
 <via x="63.119" y="11.303" extent="1-16" drill="1.016"/>
@@
 <wire x1="63.119" y1="4.699" x2="65.8495" y2="1.9685" width="0.635" layer="16"/>
 <wire x1="65.8495" y1="1.9685" x2="82.8675" y2="1.9685" width="0.635" layer="16"/>
+<contactref element="NANO" pad="13"/>
+<contactref element="JP2" pad="3"/>
+<wire x1="52.324" y1="28.575" x2="45.974" y2="28.575" width="0.635" layer="16"/>
+<wire x1="54.864" y1="26.035" x2="52.324" y2="28.575" width="0" layer="19" extent="16-16"/>
 </signal>
 <signal name="A6">
